File: DotBot-LH2-Shield.kicad_sch (KiCad schematic)
At the start: 23 parts, among them J1 Conn_01x04, J1 Conn_01x10, Q1 NX6008NBKWX, Q2 NX6008NBKWX, Q3 NX6008NBKWX, U3 ISM330DHCXTR, U4 LIS3MDL, U4 TS4231

Commit message: update BOM on the shield
Parts:
- Q1, Q2, Q3: Link (none) -> https://www.digikey.com/short/n5qrw293; Manufacturer (none) -> Nexperia USA Inc.; Mfr Part Number (none) -> NX6008NBKWX
- R1: AISLER_MPN ERA-3AEB471V -> RC0603FR-07750RL; Link https://www.digikey.fr/short/q439jwb0 -> https://www.digikey.com/short/pr59n47j; Manufacturer Panasonic Electronic Components -> YAGEO; Mfr Part Number ERA-3AEB471V -> RC0603FR-07750RL
- R2: AISLER_MPN ERJ-PB3D2610V -> RC0603FR-07750RL; Link https://www.digikey.fr/short/rj3trjhr -> https://www.digikey.com/short/pr59n47j; Manufacturer Panasonic Electronic Components -> YAGEO; Mfr Part Number ERJ-PB3D2610V -> RC0603FR-07750RL
- R3: AISLER_MPN ERJ-PB3D2400V -> CRGCQ0603F1K0; Link https://www.digikey.fr/short/ddpj9vb4 -> https://www.digikey.com/short/932zt05j; Manufacturer Panasonic Electronic Components -> TE Connectivity Passive Product; Mfr Part Number ERJ-PB3D2400V -> CRGCQ0603F1K0
Changed lines of the file:
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@@
+      (effects (font (size 1.27 1.27)) hide)
+    )
+    (property "Link" "https://www.digikey.com/short/n5qrw293" (at 189.23 54.61 0)
+      (effects (font (size 1.27 1.27)) hide)
+    )
+    (property "Manufacturer" "Nexperia USA Inc." (at 189.23 54.61 0)
+      (effects (font (size 1.27 1.27)) hide)
+    )
+    (property "Mfr Part Number" "NX6008NBKWX" (at 189.23 54.61 0)
       (effects (font (size 1.27 1.27)) hide)
     )
@@
       (effects (font (size 1.27 1.27)) hide)
     )
+    (property "Link" "https://www.digikey.com/short/n5qrw293" (at 237.49 68.58 0)
+      (effects (font (size 1.27 1.27)) hide)
+    )
+    (property "Manufacturer" "Nexperia USA Inc." (at 237.49 68.58 0)
+      (effects (font (size 1.27 1.27)) hide)
+    )
+    (property "Mfr Part Number" "NX6008NBKWX" (at 237.49 68.58 0)
+      (effects (font (size 1.27 1.27)) hide)
+    )
     (pin "1")
     (pin "2")
@@
       (effects (font (size 1.27 1.27)) hide)
     )
-    (property "Link" "https://www.digikey.fr/short/rj3trjhr" (at 240.03 44.45 0)
-      (effects (font (size 1.27 1.27)) hide)
-    )
-    (property "Manufacturer" "Panasonic Electronic Components" (at 240.03 44.45 0)
-      (effects (font (size 1.27 1.27)) hide)
-    )
-    (property "Mfr Part Number" "ERJ-PB3D2610V" (at 240.03 44.45 0)
+    (property "Link" "https://www.digikey.com/short/pr59n47j" (at 240.03 44.45 0)
+      (effects (font (size 1.27 1.27)) hide)
+    )
+    (property "Manufacturer" "YAGEO" (at 240.03 44.45 0)
+      (effects (font (size 1.27 1.27)) hide)
+    )
+    (property "Mfr Part Number" "RC0603FR-07750RL" (at 240.03 44.45 0)
       (effects (font (size 1.27 1.27)) hide)
     )
@@
       (effects (font (size 1.27 1.27)) hide)
     )
-    (property "AISLER_MPN" "ERJ-PB3D2610V" (at 240.03 44.45 0)
+    (property "AISLER_MPN" "RC0603FR-07750RL" (at 240.03 44.45 0)
       (effects (font (size 1.27 1.27)) hide)
     )
@@
       (effects (font (size 1.27 1.27)) hide)
     )
-    (property "Link" "https://www.digikey.fr/short/q439jwb0" (at 215.9 44.45 0)
-      (effects (font (size 1.27 1.27)) hide)
-    )
-    (property "Manufacturer" "Panasonic Electronic Components" (at 215.9 44.45 0)
-      (effects (font (size 1.27 1.27)) hide)
-    )
-    (property "Mfr Part Number" "ERA-3AEB471V" (at 215.9 44.45 0)
+    (property "Link" "https://www.digikey.com/short/pr59n47j" (at 215.9 44.45 0)
+      (effects (font (size 1.27 1.27)) hide)
+    )
+    (property "Manufacturer" "YAGEO" (at 215.9 44.45 0)
+      (effects (font (size 1.27 1.27)) hide)
+    )
+    (property "Mfr Part Number" "RC0603FR-07750RL" (at 215.9 44.45 0)
       (effects (font (size 1.27 1.27)) hide)
     )
@@
       (effects (font (size 1.27 1.27)) hide)
     )
-    (property "AISLER_MPN" "ERA-3AEB471V" (at 215.9 44.45 0)
+    (property "AISLER_MPN" "RC0603FR-07750RL" (at 215.9 44.45 0)
       (effects (font (size 1.27 1.27)) hide)
     )
@@
       (effects (font (size 1.27 1.27)) hide)
     )
+    (property "Link" "https://www.digikey.com/short/n5qrw293" (at 213.36 62.23 0)
+      (effects (font (size 1.27 1.27)) hide)
+    )
+    (property "Manufacturer" "Nexperia USA Inc." (at 213.36 62.23 0)
+      (effects (font (size 1.27 1.27)) hide)
+    )
+    (property "Mfr Part Number" "NX6008NBKWX" (at 213.36 62.23 0)
+      (effects (font (size 1.27 1.27)) hide)
+    )
     (pin "1")
     (pin "2")
@@
       (effects (font (size 1.27 1.27)) hide)
     )
-    (property "Link" "https://www.digikey.fr/short/ddpj9vb4" (at 191.77 44.45 0)
-      (effects (font (size 1.27 1.27)) hide)
-    )
-    (property "Manufacturer" "Panasonic Electronic Components" (at 191.77 44.45 0)
-      (effects (font (size 1.27 1.27)) hide)
-    )
-    (property "Mfr Part Number" "ERJ-PB3D2400V" (at 191.77 44.45 0)
+    (property "Link" "https://www.digikey.com/short/932zt05j" (at 191.77 44.45 0)
+      (effects (font (size 1.27 1.27)) hide)
+    )
+    (property "Manufacturer" "TE Connectivity Passive Product" (at 191.77 44.45 0)
+      (effects (font (size 1.27 1.27)) hide)
+    )
+    (property "Mfr Part Number" "CRGCQ0603F1K0" (at 191.77 44.45 0)
       (effects (font (size 1.27 1.27)) hide)
     )
@@
       (effects (font (size 1.27 1.27)) hide)
     )
-    (property "AISLER_MPN" "ERJ-PB3D2400V" (at 191.77 44.45 0)
-      (effects (font (size 1.27 1.27)) hide)
-    )
+    (property "AISLER_MPN" "CRGCQ0603F1K0" (at 191.77 44.45 0)
+      (effects (font (size 1.27 1.27)) hide)
+    )

Commit message: fix: lh2 shield BOM. Some links were to digikey.com not digikey.fr
Parts:
- Q1, Q2, Q3: Link https://www.digikey.com/short/n5qrw293 -> https://www.digikey.fr/short/t1h7z77b
- R1, R2: Link https://www.digikey.com/short/pr59n47j -> https://www.digikey.fr/short/vzftpbc3
- R3: Link https://www.digikey.com/short/932zt05j -> https://www.digikey.fr/short/752z5hbm
Changed lines of the file:
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@@
       (effects (font (size 1.27 1.27)) hide)
     )
-    (property "Link" "https://www.digikey.com/short/n5qrw293" (at 189.23 54.61 0)
+    (property "Link" "https://www.digikey.fr/short/t1h7z77b" (at 189.23 54.61 0)
       (effects (font (size 1.27 1.27)) hide)
     )
@@
       (effects (font (size 1.27 1.27)) hide)
     )
-    (property "Link" "https://www.digikey.com/short/n5qrw293" (at 237.49 68.58 0)
+    (property "Link" "https://www.digikey.fr/short/t1h7z77b" (at 237.49 68.58 0)
       (effects (font (size 1.27 1.27)) hide)
     )
@@
       (effects (font (size 1.27 1.27)) hide)
     )
-    (property "Link" "https://www.digikey.com/short/pr59n47j" (at 240.03 44.45 0)
+    (property "Link" "https://www.digikey.fr/short/vzftpbc3" (at 240.03 44.45 0)
       (effects (font (size 1.27 1.27)) hide)
     )
@@
       (effects (font (size 1.27 1.27)) hide)
     )
-    (property "Link" "https://www.digikey.com/short/pr59n47j" (at 215.9 44.45 0)
+    (property "Link" "https://www.digikey.fr/short/vzftpbc3" (at 215.9 44.45 0)
       (effects (font (size 1.27 1.27)) hide)
     )
@@
       (effects (font (size 1.27 1.27)) hide)
     )
-    (property "Link" "https://www.digikey.com/short/n5qrw293" (at 213.36 62.23 0)
+    (property "Link" "https://www.digikey.fr/short/t1h7z77b" (at 213.36 62.23 0)
       (effects (font (size 1.27 1.27)) hide)
     )
@@
       (effects (font (size 1.27 1.27)) hide)
     )
-    (property "Link" "https://www.digikey.com/short/932zt05j" (at 191.77 44.45 0)
-      (effects (font (size 1.27 1.27)) hide)
-    )
+    (property "Link" "https://www.digikey.fr/short/752z5hbm" (at 191.77 44.45 0)
+      (effects (font (size 1.27 1.27)) hide)
+    )
