File: pcb/shields/template/DotBot-Shield-Template.kicad_pcb (KiCad board)
At the start: 4 copper layers, 29 x 27 mm, 3 parts, among them J1 Bottom Header, J2 Left Header, J3 Right Header

Commit message: pcb/shields/template: fix background silkscreen labels
Other:
- board text added: "P0.02"
- board text added: "P0.03"
- board text added: "P0.10"
- board text added: "P0.11"
- board text added: "P0.27"
- board text added: "P1.01"
- board text added: "P1.06"
- board text added: "P1.07"
- board text removed: "EXT_1/P0.30"
- board text removed: "EXT_2/P0.09"
- board text removed: "P0.02/SCL"
- board text removed: "P0.03/SDA"
- board text removed: "P0.10/G"
- board text removed: "P0.11/INT"
- board text removed: "P0.27/E"
- board text removed: "P1.01/D"
- board text removed: "P1.06/R"
- board text removed: "P1.07/B"
Changed lines of the file:
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@@
   (gr_line (start 130.048 125) (end 154.94 125)
     (stroke (width 0.1) (type default)) (layer "Edge.Cuts"))
-  (gr_text "EXT_1/P0.30" (at 140.97 121.412 270) (layer "B.SilkS")
+  (gr_text "P0.30" (at 140.97 121.412 270) (layer "B.SilkS")
     (effects (font (size 0.8 0.8) (thickness 0.1875)) (justify left bottom mirror))
   )
-  (gr_text "P1.01/D" (at 136.906 103.124) (layer "B.SilkS")
+  (gr_text "P1.01" (at 135.28 103.124) (layer "B.SilkS")
     (effects (font (size 0.8 0.8) (thickness 0.1875)) (justify left bottom mirror))
   )
-  (gr_text "P1.07/B" (at 136.906 110.744) (layer "B.SilkS")
+  (gr_text "P1.07" (at 135.32 110.744) (layer "B.SilkS")
     (effects (font (size 0.8 0.8) (thickness 0.1875)) (justify left bottom mirror))
   )
-  (gr_text "P1.06/R" (at 136.906 113.284) (layer "B.SilkS")
+  (gr_text "P1.06" (at 135.28 113.284) (layer "B.SilkS")
     (effects (font (size 0.8 0.8) (thickness 0.1875)) (justify left bottom mirror))
   )
@@
     (effects (font (size 0.8 0.8) (thickness 0.1875)) (justify left bottom mirror))
   )
-  (gr_text "P0.11/INT" (at 137.668 115.824) (layer "B.SilkS")
+  (gr_text "P0.11" (at 135.28 115.86) (layer "B.SilkS")
     (effects (font (size 0.8 0.8) (thickness 0.1875)) (justify left bottom mirror))
   )
@@
     (effects (font (size 0.8 0.8) (thickness 0.1875)) (justify left bottom mirror))
   )
-  (gr_text "P0.02/SCL" (at 153.416 108.204) (layer "B.SilkS")
+  (gr_text "P0.02" (at 153.416 108.204) (layer "B.SilkS")
     (effects (font (size 0.8 0.8) (thickness 0.1875)) (justify left bottom mirror))
   )
@@
     (effects (font (size 0.8 0.8) (thickness 0.1875)) (justify left bottom mirror))
   )
-  (gr_text "P0.27/E" (at 136.906 105.664) (layer "B.SilkS")
+  (gr_text "P0.27" (at 135.35 105.664) (layer "B.SilkS")
     (effects (font (size 0.8 0.8) (thickness 0.1875)) (justify left bottom mirror))
   )
@@
     (effects (font (size 0.8 0.8) (thickness 0.1875)) (justify left bottom mirror))
   )
-  (gr_text "P0.10/G" (at 136.906 108.204) (layer "B.SilkS")
+  (gr_text "P0.10" (at 135.32 108.204) (layer "B.SilkS")
     (effects (font (size 0.8 0.8) (thickness 0.1875)) (justify left bottom mirror))
   )
-  (gr_text "EXT_2/P0.09" (at 143.51 121.412 270) (layer "B.SilkS")
+  (gr_text "P0.09" (at 143.51 121.412 270) (layer "B.SilkS")
     (effects (font (size 0.8 0.8) (thickness 0.1875)) (justify left bottom mirror))
   )
@@
     (effects (font (size 0.8 0.8) (thickness 0.1875)) (justify left bottom mirror))
   )
-  (gr_text "P0.03/SDA" (at 153.416 105.664) (layer "B.SilkS")
+  (gr_text "P0.03" (at 153.416 105.664) (layer "B.SilkS")
     (effects (font (size 0.8 0.8) (thickness 0.1875)) (justify left bottom mirror))
   )
