File: pcb/DotBot.kicad_sch (KiCad schematic)
At the start: 52 parts, among them J1 Left Shield Header, J10 Extra Pins, J11 Motor connector, J12 Motor connector, J6 SWD, J7 Right Shield Header, J8 Extra Pins, J9 Extra Pins, Q1 NX6008NBKWX, Q2 NX6008NBKWX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

Commit message: #11 3v-motor: update BOM in schematic
Parts:
- BT1: Price 0.833 -> 0.932
- C10: Price 0.004 -> 0.005
- C18, C19: Price 0.0085 -> 0.0043
- C3, C4: Manufacturer (none) -> Samsung Electro-Mechanics
- C9: Link https://www.digikey.fr/short/84p7mf1t -> https://www.digikey.fr/short/pm3hbfq0; Manufacturer (none) -> Samsung Electro-Mechanics; Mfr Part Number CGA3E2X7R1H103K080AA -> CL10B104KB8NNWC; Price 0.013 -> 0.005
- D1: Price 0.146 -> 0.176
- J11, J12: Price 0.067 -> 0.079
- L2: Price 0.127 -> 0.11
- LD1, LD2: Price 0.062 -> 0.066
- Q1, Q2, Q5: Price (none) -> 0.043
- Q3, Q4: Manufacturer (none) -> Diodes Incorporated; Price 0.10 -> 0.097
- R1: Link https://www.digikey.com/short/vj5058q2 -> https://www.digikey.com/short/9tvpdt8v; Manufacturer (none) -> YAGEO; Mfr Part Number RC0603FR-071RL -> RC0603FR-07220KL; Price 0.0087 -> 0.0055
- R12, R13, R14: Link https://www.digikey.fr/short/fr3tftdj -> https://www.digikey.com/short/5whqz3bv; Manufacturer (none) -> YAGEO; Mfr Part Number YAG3561TR-ND -> RC0603FR-07100RL; Price 0.006 -> 0.0053
- R2, R3: Link https://www.digikey.com/short/vj5058q2 -> https://www.digikey.com/short/t40bvh3q; Manufacturer (none) -> Stackpole Electronics Inc; Mfr Part Number RC0603FR-071RL -> RMCF0603FT6K19; Price 0.0087 -> 0.00425
- R4: Link https://www.digikey.com/short/vj5058q2 -> https://www.digikey.com/short/dt0m9h2r; Manufacturer (none) -> YAGEO; Mfr Part Number RC0603FR-071RL -> RC0603FR-131ML; Price 0.0087 -> 0.0053
- R5: AISLER_MPN CRGCQ0603F1K0 -> (none); Link https://www.digikey.fr/short/752z5hbm -> https://www.digikey.com/short/w9nhv25z; Manufacturer TE Connectivity Passive Product -> YAGEO; Mfr Part Number CRGCQ0603F1K0 -> RC0603FR-07750RL; Price 0.19 -> 0.0053
- R6: AISLER_MPN RC0603FR-07750RL -> (none); Link https://www.digikey.fr/short/vzftpbc3 -> https://www.digikey.com/short/f3rj09jr; Mfr Part Number RC0603FR-07750RL -> RC0603FR-10510RL; Price 0.35 -> 0.0055
- R7: AISLER_MPN RC0603FR-07750RL -> (none); Link https://www.digikey.fr/short/vzftpbc3 -> https://www.digikey.com/short/f3rj09jr; Mfr Part Number RC0603FR-07750RL -> RC0603FR-10510RL; Price 0.19 -> 0.0055
- SW1: Price 0.568 -> 0.654
- U1, U2, U4, U5: Price 0.25 -> 0.299
- U6: Link (none) -> https://www.digikey.com/short/p5zn27bv; Mfr Part Number (none) -> DRV8411ARTER; Price (none) -> 1.11
- U7: Price 9.97 -> 8.70
- U8: Link (none) -> https://www.digikey.fr/short/vfjcbbq3; Manufacturer (none) -> Analog Devices Inc./Maxim Integrated; Mfr Part Number (none) -> MAX1724EZK50+T; Price (none) -> 2.36
- U9: Manufacturer (none) -> Analog Devices Inc.; Mfr Part Number 505-ADP121-AUJZ33R7TR-ND -> ADP121-AUJZ33R7; Price 0.626 -> 0.59
