File: pcb/shields/lh2/DotBot-LH2-Shield.kicad_sch (KiCad schematic)
At the start: 23 parts, among them J1 Conn_01x04, J1 Conn_01x10, Q1 NX6008NBKWX, Q2 NX6008NBKWX, Q3 NX6008NBKWX, U3 ISM330DHCXTR, U4 LIS3MDL, U4 TS4231

Commit message: doc: update BOM prices
Parts:
- C1, C3, C4, C9: Price 0.004 -> 0.0046; now not fitted
- C2, C4: Price 0.007 -> 0.0077; now not fitted
- D1: Price 0.49 -> 0.40; now not fitted
- D2: Price 0.146 -> 0.175; now not fitted
- Q1, Q2, Q3: Price (none) -> 0.042; now not fitted
- R1: Price 0.35 -> 0.005; now not fitted
- R2: Price 0.0043 -> 0.0053; now not fitted
- R2: Price 0.19 -> 0.005; now not fitted
- R3: Price 0.19 -> 0.007; now not fitted
- U3: Price 11.34 -> 4.98; now not fitted
- U4: Price 0.945 -> 0.787; now not fitted
- U4: Price 1.962 -> 2.12

Commit message: fix: remove accidental DNP marks
Parts:
- C1, C2, C3, C4, C9, D1, D2, Q1, Q2, Q3, R1, R2, R3, U3, U4: now fitted
Changed lines of the file:
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@@
 		(in_bom yes)
 		(on_board yes)
-		(dnp yes)
+		(dnp no)
 		(property "Reference" "C4"
 			(at 181.61 96.52 0)
@@
 		(in_bom yes)
 		(on_board yes)
-		(dnp yes)
+		(dnp no)
 		(property "Reference" "D2"
 			(at 186.69 27.94 90)
@@
 		(in_bom yes)
 		(on_board yes)
-		(dnp yes)
+		(dnp no)
 		(property "Reference" "C3"
 			(at 85.09 96.52 0)
@@
 		(in_bom yes)
 		(on_board yes)
-		(dnp yes)
+		(dnp no)
 		(property "Reference" "R2"
 			(at 138.43 60.96 90)
@@
 		(in_bom yes)
 		(on_board yes)
-		(dnp yes)
+		(dnp no)
 		(property "Reference" "D1"
 			(at 83.82 64.77 90)
@@
 		(in_bom yes)
 		(on_board yes)
-		(dnp yes)
+		(dnp no)
 		(property "Reference" "C4"
 			(at 96.52 96.52 0)
@@
 		(in_bom yes)
 		(on_board yes)
-		(dnp yes)
+		(dnp no)
 		(property "Reference" "U4"
 			(at 123.19 44.45 0)
@@
 		(in_bom yes)
 		(on_board yes)
-		(dnp yes)
+		(dnp no)
 		(property "Reference" "Q1"
 			(at 195.58 53.34 0)
@@
 		(in_bom yes)
 		(on_board yes)
-		(dnp yes)
+		(dnp no)
 		(property "Reference" "C4"
 			(at 172.72 96.52 0)
@@
 		(in_bom yes)
 		(on_board yes)
-		(dnp yes)
+		(dnp no)
 		(property "Reference" "Q3"
 			(at 243.84 67.31 0)
@@
 		(in_bom yes)
 		(on_board yes)
-		(dnp yes)
+		(dnp no)
 		(property "Reference" "R2"
 			(at 242.57 44.45 90)
@@
 		(in_bom yes)
 		(on_board yes)
-		(dnp yes)
+		(dnp no)
 		(property "Reference" "C9"
 			(at 220.98 22.86 0)
@@
 		(in_bom yes)
 		(on_board yes)
-		(dnp yes)
+		(dnp no)
 		(property "Reference" "C2"
 			(at 92.71 55.88 90)
@@
 		(in_bom yes)
 		(on_board yes)
-		(dnp yes)
+		(dnp no)
 		(property "Reference" "C4"
 			(at 217.17 123.19 0)
@@
 		(in_bom yes)
 		(on_board yes)
-		(dnp yes)
+		(dnp no)
 		(property "Reference" "R1"
 			(at 218.44 44.45 90)
@@
 		(in_bom yes)
 		(on_board yes)
-		(dnp yes)
+		(dnp no)
 		(property "Reference" "Q2"
 			(at 219.71 60.96 0)
@@
 		(in_bom yes)
 		(on_board yes)
-		(dnp yes)
+		(dnp no)
 		(property "Reference" "R3"
 			(at 194.31 44.45 90)
@@
 		(in_bom yes)
 		(on_board yes)
-		(dnp yes)
+		(dnp no)
 		(property "Reference" "U3"
 			(at 99.06 129.54 0)
@@
 		(in_bom yes)
 		(on_board yes)
-		(dnp yes)
+		(dnp no)
 		(property "Reference" "C1"
 			(at 92.71 49.53 90)
